File: KiCad/TPA2016+UDA1334/TPA2016+UDA1334.kicad_sch (KiCad schematic)
At the start: 33 parts, among them U1 UDA1334ATS, U2 MIC5225-3.3

Commit message: started work on combining the two schematics
Parts:
- removed U1: UDA1334ATS, Package_SO:HTSSOP-16-1EP_4.4x5mm_P0.65mm_EP3.4x5mm, symbol UDA1334-eagle-import:AUDIO_I2S_UDA1334{dblquote}{dblquote}
- added U?: UDA1334ATS, Package_SO:SSOP-16_4.4x5.2mm_P0.65mm, symbol Audio:UDA1334ATS
Connections:
- net 3.3V: now also U?.4 (VDDD)
- net BITCLK_IN: now also U?.1 (BCK)
- net DATA_IN: now also U?.3 (DATAI)
- net DEEM/CLKOUT: now also U?.9 (DEEM/CLKOUT)
- net GND: now also U?.5 (VSSD)
- net GNDA: now also U?.15 (VSSA)
- net MUTE: now also U?.8 (MUTE)
- net PLL_IN: now also U?.10 (PLL0)
- net SFOR0: now also U?.11 (SFOR0)
- net SFOR1: now also U?.7 (SFOR1)
- net SYSCLK_IN: now also U?.6 (SYSCLK/PLL1)
- net WORDSEL_IN: now also U?.2 (WS)
- net VDDA: now reaches C1.1, C2.1, FB1.1
- net VDDA: now also U?.13 (VDDA)
- net at C5.1, C9.1: now also U?.12 (Vref(DAC))
- net at C6.1: now also U?.14 (VOUTL)
- net at C10.1: now also U?.16 (VOUTR)
Other:
- note added: "UDA1334"
- moved on the sheet: C1, C10, C11, C12, C121, C2, C3, C4, C5, C6, C7, C8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

Commit message: actually combined both board schematics, need to do more tho
Parts:
- added C1, C9: 10µF, Capacitor_SMD:C_0805_2012Metric, symbol Device:C_Small
- added C2, C3, C4: 0.1µF, Capacitor_SMD:C_0805_2012Metric, symbol Device:C_Small
- added C5, C6, C7, C8: 1µF, Capacitor_SMD:C_0805_2012Metric, symbol Device:C_Small
- added FB1, FB2: ferrite, Resistor_SMD:R_0805_2012Metric, symbol Device:FerriteBead_Small
- added IC1: TPA2016D2QFN, Package_DFN_QFN:QFN-20-1EP_4x4mm_P0.5mm_EP2.5x2.5mm, symbol TPA2016D2-eagle-import:TPA2016D2QFN
- added J1, J2: TERMBLOCK_1X2, Connector_PinHeader_2.54mm:PinHeader_1x02_P2.54mm_Vertical, symbol Connector_Generic:Conn_01x02
- added JP1: HEADER-1X10, Connector_PinHeader_2.54mm:PinHeader_1x10_P2.54mm_Vertical, symbol Connector_Generic:Conn_01x10
- added R1, R2: 10K, Capacitor_SMD:C_0805_2012Metric, symbol Device:R_Small
- added R3: 100K, Capacitor_SMD:C_0805_2012Metric, symbol Device:R_Small
- added U$20, U$21: MOUNTINGHOLE, MountingHole:MountingHole_2.2mm_M2, symbol Mechanical:MountingHole
Connections:
- net GND: now also C1.2, C3.1, C4.2, C9.2, FB2.1, IC1.21 (THERMAL), IC1.8 (PGND), JP1.2 (Pin_2)
- net GNDA: now also C2.2, C3.2, FB2.2, IC1.3 (AGND)
- net VDDA: now also C2.1, FB1.2, IC1.13 (AVDD)
- new net: C5.2, IC1.2 (INL-)
- new net: C8.2, IC1.14 (INR-)
- new net: C6.2, IC1.1 (INL+)
- new net: C7.2, IC1.15 (INR+)
- new net I2C_VCC: JP1.10 (Pin_10), R1.2, R2.2
- new net IN_L_N: C5.1, JP1.7 (Pin_7)
- new net IN_L_P: C6.1, JP1.6 (Pin_6)
- new net IN_R_N: C8.1, JP1.4 (Pin_4)
- new net IN_R_P: C7.1, JP1.5 (Pin_5)
- new net OUT_L_N: IC1.7 (OUTL-), J1.1 (Pin_1)
- new net OUT_L_P: IC1.6 (OUTL+), J1.2 (Pin_2)
- new net OUT_R_N: IC1.9 (OUTR-), J2.2 (Pin_2)
- new net OUT_R_P: IC1.10 (OUTR+), J2.1 (Pin_1)
- new net SCL: IC1.17 (SCL), JP1.8 (Pin_8), R1.1
- new net SDA: IC1.19 (SDA), JP1.9 (Pin_9), R2.1
- new net SHUTDOWN: IC1.18 (SDZ), JP1.3 (Pin_3), R3.1
- new net VDD: C1.1, C4.1, C9.1, FB1.1, IC1.11 (PVDDR@1), IC1.12 (PVDDR@2), IC1.4 (PVDDL@1), IC1.5 (PVDDL@2), JP1.1 (Pin_1), R3.2
Other:
- note added: "Any resistance or inductance in the trace"
- note added: "Note on speaker choice (4/8/16/32 ohm, etc.):"
- note added: "Place C1 as close as possible to PVDD."
- note added: "TPA2016D2QFN"
- note added: "The audio input pins (INR+/-"
- note added: "Using speakers more resistive than 4-Ω"
- note added: "and INL+/-) must run"
- note added: "between the device and the capacitor can"
- note added: "by reducing the output current and increasing"
- note added: "cause a loss in efficiency"
- note added: "common-mode noise cancellation."
- note added: "dramatically increases the thermal performance"
- note added: "side-by-side to maximize"
- note added: "the efficiency of the amplifier."
- moved on the sheet: C1, C10, C11, C12, C121, C2, C3, C4, C5, C6, C7, C8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
