File: KiCad/USB-Sound-Card/PCM2900C.kicad_sch (KiCad schematic)
At the start: 21 parts, among them J101 USB_C_Receptacle_USB2.0, J2 Conn_01x03_Male, U101 PCM2900C, Y1 12MHz 18pF

Commit message: hastily slapped together pcb
Parts:
- removed J2: Conn_01x03_Male, Connector_PinHeader_2.54mm:PinHeader_1x03_P2.54mm_Vertical, symbol Connector_Generic:Conn_01x03
- added J102: AudioJack3, Connector_Audio:Jack_3.5mm_CUI_SJ1-3523N_Horizontal, symbol Connector:AudioJack3
- C10, C11, C12, C13, C14, C15, C16, C6, C7, C8, C9: footprint Capacitor_SMD:C_0805_2012Metric -> Capacitor_SMD:C_0402_1005Metric
- R1, R101, R102, R2: footprint Resistor_SMD:R_0805_2012Metric -> Resistor_SMD:R_0402_1005Metric
Connections:
- net AGNDC: now also J102.S
- net L-USB-In: now also J102.T
- net R-USB-In: now also J102.R

Commit message: added some amps, may change
Parts:
- removed J102: AudioJack3, Connector_Audio:Jack_3.5mm_CUI_SJ1-3523N_Horizontal, symbol Connector:AudioJack3
- added C? (x2): 10µF, Capacitor_SMD:C_0402_1005Metric, symbol Device:C
- added C? (x2): 1µF, Capacitor_SMD:C_0402_1005Metric, symbol Device:C
- added U? (x2): PAM8302AAD, Package_SO:Diodes_SO-8EP, symbol Amplifier_Audio:PAM8302AAD
Connections:
- net AGNDC: now also U?.4 (IN-), U?.4 (IN-)
- net GNDD: now also C?.1, C?.1, C?.2, C?.2, U?.7 (GND), U?.7 (GND)
- net L-USB-In: now also U?.3 (IN+)
- net R-USB-In: now also U?.3 (IN+)
- net VBUS: now also C?.1, C?.1, C?.2, C?.2, U?.6 (VDD), U?.6 (VDD)
Other:
- moved on the sheet: C10, C11, C12, C13, C14, C15, C16, C6, C9, R1, R2, U101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

Commit message: some general board design progress and rearrangement, need to re-do bits of the board still
Parts:
- added H1, H2, H3, H4: MountingHole, MountingHole:MountingHole_2.2mm_M2, symbol Mechanical:MountingHole
- added J1, J2: MPT 2.54, TerminalBlock_Phoenix:TerminalBlock_Phoenix_MPT-0,5-2-2.54_1x02_P2.54mm_Horizontal, symbol Connector_Generic:Conn_01x02
- added J3, J4: TestPoint, TestPoint:TestPoint_Pad_1.0x1.0mm, symbol Connector_Generic:Conn_01x01
- C1, C3: renamed from C?; value 10µF -> 10µF 0402
- C10, C11, C12, C13, C14, C9: value 1µF -> 1µF 0402
- C15, C16: value 22pF -> 22pF 0402
- C2, C4: renamed from C?; value 1µF -> 1µF 0402
- C6, C7, C8: value 10µF -> 10µF 0402
- R1: value 1M -> 1M 0402
- R101, R102: value 5.1K 0805 -> 5.1K 0402
- R2: value 2R2 -> 2R2 0402
- Y1: value 12MHz 18pF -> 12MHz 18pF 3225-4P
- gave numbers to parts that had none: 2
Connections:
- net at U1.1 (~{SD}): now also J3.1 (Pin_1)
- net at U1.5 (OUT+): now also J1.1 (Pin_1)
- net at U1.8 (OUT-): now also J1.2 (Pin_2)
- net at U2.1 (~{SD}): now also J4.1 (Pin_1)
- net at U2.5 (OUT+): now also J2.1 (Pin_1)
- net at U2.8 (OUT-): now also J2.2 (Pin_2)
Other:
- moved on the sheet: C1, C10, C11, C12, C13, C14, C15, C16, C2, C3, C4, C6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
