File: KiCad/EnvOpenAudio/EnvOpenAudio.kicad_pcb (KiCad board)
At the start: 2 copper layers, 21 x 51 mm, 58 parts, among them J2 Button, J3 2.54mm header 01x20, J4 2.54mm header 01x20, J5 Conn_01x03_Male, Q1 SI2301B, U1 SOT-23-5 5.5V 3.3V 500mA, U3 RP2040, Y1 3225_4P 12MHz

Commit message: started work on RP2040 board
Parts:
- removed GP23_LED1: GP23 LED_0402, LED_SMD:LED_0402_1005Metric
- removed GPIO24_RESISTOR1: 1K 0402, Resistor_SMD:R_0402_1005Metric
- removed GPIO25_LED1: LED_0402, LED_SMD:LED_0402_1005Metric
- removed GPIO25_RESISTOR1: 470 0402, Resistor_SMD:R_0402_1005Metric
- removed J3, J4: 2.54mm header 01x20, Connector_PinHeader_2.54mm:PinHeader_1x20_P2.54mm_Vertical
- removed Q1: SI2301B, Package_TO_SOT_SMD:SOT-23
- removed REF**: OSHW-Symbol_6.7x6mm_Copper, Symbol:OSHW-Symbol_6.7x6mm_Copper
- removed REF**: Symbol_GNU-GPL_CopperTop_Small, Symbol:Symbol_GNU-GPL_CopperTop_Small
- removed REF**: KiCad-Logo2_5mm_SilkScreen, Symbol:KiCad-Logo2_5mm_SilkScreen
- removed USB1: TYPE-C-31-M-12, HRO-TYPE-C31-M-12:HRO-TYPE-C-31-M-12
- added J1: USB_C_Receptacle_USB2.0, Connector_USB:USB_C_Receptacle_HRO_TYPE-C-31-M-12, F.Cu at (103.7, 60.9)
- J5: footprint Connector_PinHeader_2.54mm:PinHeader_1x03_P2.54mm_Vertical -> Connector_PinHeader_1.00mm:PinHeader_1x03_P1.00mm_Vertical
- moved J5 8.19 mm to (102.3, 98.8)
Routing:
- net /GPIO23: track 31.5 -> 0.00 mm, vias 2 -> 0
- net /GPIO0: track 28.5 -> 0.00 mm
- net Net-(GPIO25_LED1-A): track 26.7 -> 0.00 mm, vias 2 -> 0
- net /GPIO1: track 26.4 -> 0.00 mm
- net /GPIO2: track 21.8 -> 0.00 mm
- net /GPIO3: track 21.3 -> 0.00 mm, vias 1 -> 0
- net /GPIO15: track 23.5 -> 2.91 mm
- net /GPIO16: track 20.2 -> 0.00 mm
- net GND: track 43.5 -> 23.3 mm
- net /GPIO4: track 20.0 -> 0.00 mm, vias 1 -> 0
- net /GPIO14: track 18.5 -> 0.00 mm
- net /GPIO5: track 17.8 -> 0.00 mm, vias 1 -> 0
- net /GPIO17: track 17.6 -> 0.00 mm
- net /SWCLK: track 28.9 -> 12.3 mm
- net /GPIO13: track 14.0 -> 0.00 mm
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Other:
- board text added: "#REV 1.0"
- board text added: "EnvOpenAudio"
- board text removed: "#REV 1.4"
- board text removed: "19"
- board text removed: "20"
- board text removed: "23"
- board text removed: "25"
- board text removed: "3V3"
- board text removed: "3V3EN"
- board text removed: "4"
- board text removed: "5"
- board text removed: "6"
- board text removed: "7"
- board text removed: "AGND"
- board text removed: "BOOT"
- board text removed: "BOOTSEL"
- board text removed: "CBP1"
- board text removed: "D+"
- board text removed: "D-"
- board text removed: "EnvOpenPico"
- board text removed: "G"
- board text removed: "GND"
- board text removed: "GP0"
- board text removed: "GP1"
- board text removed: "GP10"
- board text removed: "GP11"
- board text removed: "GP12"
- board text removed: "GP13"
- board text removed: "GP14"
- board text removed: "GP15"
- board text removed: "GP16"
- board text removed: "GP17"
- board text removed: "GP18"
- board text removed: "GP19"
- board text removed: "GP2"
- board text removed: "GP20"
- board text removed: "GP21"
- board text removed: "GP22"
- board text removed: "GP24"
- board text removed: "GP26"
- board text removed: "GP27"
- board text removed: "GP28"
- board text removed: "GP3"
- board text removed: "GP4"
- board text removed: "GP5"
- board text removed: "GP6"
- board text removed: "GP7"
- board text removed: "GP8"
- board text removed: "GP9"
- board text removed: "RESET"
- board text removed: "RUN"
- board text removed: "SWCLK"
- board text removed: "SWDIO"
- board text removed: "VBUS"
- board text removed: "VRF"
- board text removed: "VSYS"
- board text removed: "https://github.com/Envious-Data/EnvOpenPico"
