File: KiCad/EnvOpenAudio-RP2040/EnvOpenAudio.kicad_pcb (KiCad board)
At the start: 2 copper layers, 21.3 x 68.7 mm, 62 parts, among them J1 USB_C_Receptacle_USB2.0, J2 SM03B-SRSS-TB, J3 Conn_01x10, SW1 B3U-1000, SW2 B3U-1000, U1 W25Q16JVUXIQ, U2 TPS63001DRCR, U3 TLV75518PDBV, U4 RP2040, U5 TLV320AIC3100, Y1 12Mhz 2520 18pF

Commit message: few small changes, still need help with firmware.
Parts:
- added J4: Conn_01x04, Connector_PinHeader_2.54mm:PinHeader_1x04_P2.54mm_Vertical, F.Cu at (56.9, 47.6)
- C14: value 4.7uf 0402 -> 100nF
- C15, C17: value 100nf 0402 -> 1uF 0402
- U5: value TLV320AIC3100 -> TLV320AIC3110
Connections:
- J3 pad 10: unconnected-(J3-Pin_10-Pad10) -> GND
- U4 pad 19: unconnected-(U4-TESTEN-Pad19) -> GND
Routing:
- net +1V8: track 6.75 -> 48.6 mm, vias 2 -> 3
- net +3V3: track 71.5 -> 86.2 mm
- net VBUS: track 28.7 -> 34.1 mm
- net GND: track 32.3 -> 35.2 mm, vias 27 -> 28
Other:
- board text added: "3V3 1V8"
- board text added: "GND"
- board text added: "GPIO1 MIC1LP SPKP HPLO GND"
- board text removed: "GPIO1 MIC1LP SPKP HPLO NC"
