File: KiCad/EnvOpenAudio-RP2040/EnvOpenAudio.kicad_sch (KiCad schematic)
At the start: 65 parts, among them J1 USB_C_Receptacle_USB2.0, J2 SM03B-SRSS-TB, J3 Conn_01x10, SW1 B3U-1000, SW2 B3U-1000, U1 W25Q16JVUXIQ, U2 TPS63001DRCR, U3 TLV75518PDBV, U4 RP2040, U5 TLV320AIC3100, U6 LM3880, Y1 12Mhz 2520 18pF

Commit message: few small changes, still need help with firmware.
Parts:
- added J4: Conn_01x04, Connector_PinHeader_2.54mm:PinHeader_1x04_P2.54mm_Vertical, symbol Connector_Generic:Conn_01x04
- U5: value TLV320AIC3100 -> TLV320AIC3110
Connections:
- net +1V8: now also J4.2 (Pin_2)
- net +3V3: now also J4.3 (Pin_3)
- net GND: now also J3.10 (Pin_10), J4.1 (Pin_1)
- net VBUS: now also J4.4 (Pin_4)
